File: rp2354a_micro_devboard.kicad_sch (KiCad schematic)
At the start: 75 parts, among them J1 BAT+, J2 BAT-, J3 USB_C_Receptacle_USB2.0_16P, J4 01x20_PinHeader_P2.54mm, J5 01x20_PinHeader_P2.54mm, J6 SWD_SH_3p, Q1 AO3407A, Q2 AO3407A, SW1 HX_MINI_MSK12CO2, SW2 SW_SPST, SW3 SW_SPST, U1 TMI3112H, U2 MCP73832-2-OT, U4 RP2354A, U5 USBLC6-2SC6, U6 TPS613222ADBV, Y1 YIC 12M10PB

Commit message: rev0.5の完成とSK6805の削除
Parts:
- removed C14, C15, C16, C17, C21: 100n, Capacitor_SMD:C_0402_1005Metric, symbol Device:C
- removed D4, D5, D6, D7: SK6805, LED_SMD:LED_SK6805_PLCC4_2.4x2.7mm_P1.3mm, symbol LED:SK6805
- removed J4, J5: 01x20_PinHeader_P2.54mm, Connector_PinHeader_2.54mm:PinHeader_1x20_P2.54mm_Vertical, symbol Connector:Conn_01x20_Pin
- removed J6: SWD_SH_3p, Connector_JST:JST_SH_BM03B-SRSS-TB_1x03-1MP_P1.00mm_Vertical, symbol Connector:Conn_01x03_Pin
- removed R10, R11: 330, Resistor_SMD:R_0402_1005Metric, symbol Device:R
- removed SW2, SW3: SW_SPST, symbol Switch:SW_SPST
- added C19: 100n, Capacitor_SMD:C_0402_1005Metric, symbol Device:C
- added J2: Micro-DevBoard, Download_Lib:Micro-DevBoard, symbol Download_Lib:Micro-DevBoard
- added J3: SWDIO, Connector_JST:JST_SH_BM03B-SRSS-TB_1x03-1MP_P1.00mm_Vertical, symbol Connector:Conn_01x03_Pin
- added SW1, SW2: EVPAWCD40, Download_Lib:SW_SPST_EVPAW, symbol Switch:SW_Push
- C23: renamed from C13; footprint Capacitor_SMD:C_0603_1608Metric -> Capacitor_SMD:C_0402_1005Metric
- C24: renamed from C10; footprint Capacitor_SMD:C_0603_1608Metric -> Capacitor_SMD:C_0402_1005Metric
- C25: renamed from C19; footprint Capacitor_SMD:C_0603_1608Metric -> Capacitor_SMD:C_0402_1005Metric
- C3: renamed from C20; footprint Capacitor_SMD:C_0603_1608Metric -> Capacitor_SMD:C_0402_1005Metric
- C4: renamed from C24; footprint Capacitor_SMD:C_0603_1608Metric -> Capacitor_SMD:C_0402_1005Metric
- C8: renamed from C23; footprint Capacitor_SMD:C_0603_1608Metric -> Capacitor_SMD:C_0402_1005Metric
- C9: renamed from C25; footprint Capacitor_SMD:C_0603_1608Metric -> Capacitor_SMD:C_0402_1005Metric
- D1: value SS32 -> SS2040FL; footprint Diode_SMD:D_SMA -> PCM_Diode_SMD_AKL:D_SOD-123F
- Q1, Q2: footprint PCM_Package_TO_SOT_SMD_AKL:SOT-23 -> Package_TO_SOT_SMD:SOT-23
- Y1: value YIC 12M10PB -> YE12MUBCE2O; footprint Crystal:Crystal_SMD_3225-4Pin_3.2x2.5mm -> Crystal:Crystal_SMD_2016-4Pin_2.0x1.6mm
- renumbered C26 to C1, C2 to C10, C3 to C11, C4 to C12, C5 to C13, C6 to C14, C7 to C15, C8 to C17, C9 to C18, C27 to C2, C28 to C26, C11 to C27, C12 to C28, C1 to C5, C18 to C6, C22 to C7, D2 to D4, D3 to D7, J3 to J1, J1 to J4, J2 to J5, L3 to L1, L1 to L2, L2 to L3, R13 to R1, R7 to R10, R1 to R12, R5 to R14, R9 to R15, R6 to R16, R8 to R17, R16 to R2, R14 to R3, R15 to R4, R17 to R5, R12 to R6, R2 to R7, R4 to R8, R3 to R9, SW1 to SW3, U5 to U1, U4 to U2, U1 to U3, U2 to U4, U6 to U5
Connections:
- net +3V3: now also C19.1, J2.23 (Pin_23)
- net BAT_CELL: now also U4.3 (V_{BAT}); no longer U4.1 (STAT)
- net GND: now also C11.2, C12.2, C13.2, C14.2, C15.2, C17.2, C18.2, C25.2, R15.1, C19.2, J2.1 (Pin_1), J2.11 (Pin_11), J2.16 (Pin_16), J2.22 (Pin_22), J2.26 (Pin_26), J2.31 (Pin_31), J2.36 (Pin_36), J2.6 (Pin_6), J3.2 (Pin_2)
- net GPIO0: now also J2.2 (Pin_2)
- net GPIO1: now also J2.3 (Pin_3)
- net GPIO10: now also J2.14 (Pin_14)
- net GPIO11: now also J2.15 (Pin_15)
- net GPIO12: now also J2.17 (Pin_17)
- net GPIO13: now also J2.18 (Pin_18)
- net GPIO14: now also J2.19 (Pin_19)
- net GPIO15: now also J2.20 (Pin_20)
- net GPIO16: now also J2.40 (Pin_40)
- net GPIO17: now also J2.39 (Pin_39)
- net GPIO18: now also J2.38 (Pin_38)
- net GPIO19: now also J2.37 (Pin_37)
- net GPIO2: now also J2.4 (Pin_4)
- net GPIO20: now also J2.35 (Pin_35)
- net GPIO21: now also J2.34 (Pin_34)
- net GPIO22: now also J2.33 (Pin_33)
- net GPIO23: now also J2.32 (Pin_32)
- net GPIO24: now also J2.30 (Pin_30)
- net GPIO25: now also J2.29 (Pin_29)
- net GPIO26: now also J2.28 (Pin_28)
- net GPIO27: now also J2.27 (Pin_27)
- net GPIO28: now also J2.25 (Pin_25)
- net GPIO29: now also J2.24 (Pin_24)
- net GPIO3: now also J2.5 (Pin_5)
- net GPIO4: now also J2.7 (Pin_7)
- net GPIO5: now also J2.8 (Pin_8)
- net GPIO6: now also J2.9 (Pin_9)
- net GPIO7: now also J2.10 (Pin_10)
- net GPIO8: now also J2.12 (Pin_12)
- net GPIO9: now also J2.13 (Pin_13)
- net IO_VBUS: now also J2.21 (Pin_21)
- net SWCLK: now also J3.3 (Pin_3)
- net SWDIO: now also J3.1 (Pin_1)
- net +1V1: now reaches C6.1, C7.1, C8.1, C9.1, U2.23 (DVDD), U2.39 (DVDD), U2.50 (VREG_FB), U2.6 (DVDD)
- net +1V1: now also L1.1; no longer L1.2
- net at R17.2: now also U4.1 (STAT); no longer U4.3 (V_{BAT})
- net at R2.2: now also SW2.1
- net at U2.48 (VREG_LX): now also L1.2; no longer L1.1
- net at R1.2: now also SW1.1
- net at U2.26 (RUN): now also SW1.2
- net at U2.60 (~{QSPI_SS}): now also SW2.2
- no-connect marks 8 -> 7
Other:
- note removed: "for QSPI_IOVDD"
- moved on the sheet: D4, L1, R12

Commit message: fix: TPS613222 after diode OR cir
Parts:
- added D2: RB521S-30, PCM_Diode_SMD_AKL:D_SOD-523, symbol PCM_Diode_Schottky_AKL:RB521S-30
Connections:
- net IO_VBUS: now also D2.1 (K); no longer C27.1, C28.1, U5.4 (VOUT)
- new net: C27.1, C28.1, D2.2 (A), U5.4 (VOUT)
Changed lines of the file:
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@@
 	)
 	(junction
-		(at 92.71 30.48)
+		(at 248.92 30.48)
 		(diameter 0)
 		(color 0 0 0 0)
 	)
 	(junction
-		(at 243.84 30.48)
+		(at 92.71 30.48)
 		(diameter 0)
 		(color 0 0 0 0)
 	)
 	(junction
-		(at 121.92 40.64)
+		(at 243.84 30.48)
 		(diameter 0)
 		(color 0 0 0 0)
 	)
 	(junction
-		(at 52.07 45.72)
+		(at 121.92 40.64)
 		(diameter 0)
 		(color 0 0 0 0)
 	)
 	(junction
-		(at 248.92 30.48)
+		(at 52.07 45.72)
 		(diameter 0)
 		(color 0 0 0 0)
@@
 	(wire
 		(pts
-			(xy 248.92 30.48) (xy 250.19 30.48)
-		)
-		(stroke
-			(width 0)
-			(type default)
-		)
-	)
-	(wire
-		(pts
 			(xy 48.26 86.36) (xy 48.26 87.63)
 		)
@@
 	(wire
 		(pts
+			(xy 248.92 30.48) (xy 250.19 30.48)
+		)
+		(stroke
+			(width 0)
+			(type default)
+		)
+	)
+	(wire
+		(pts
 			(xy 201.93 41.91) (xy 203.2 41.91)
 		)
@@
 	(global_label "IO_VBUS"
 		(shape input)
-		(at 250.19 30.48 0)
+		(at 257.81 30.48 0)
 		(fields_autoplaced yes)
 		(effects
@@
 		)
 		(property "Intersheetrefs" "${INTERSHEET_REFS}"
-			(at 260.9767 30.48 0)
+			(at 268.5967 30.48 0)
 			(effects
 				(font
@@
 			)
 		)
+	)
+	(symbol
+		(lib_id "PCM_Diode_Schottky_AKL:RB521S-30")
+		(at 254 30.48 0)
+		(unit 1)
+		(exclude_from_sim no)
+		(in_bom yes)
+		(on_board yes)
+		(dnp no)
+		(fields_autoplaced yes)
+		(property "Reference" "D2"
+			(at 254.3175 24.13 0)
+			(effects
+				(font
+					(size 1.27 1.27)
+				)
+			)
+		)
+		(property "Value" "RB521S-30"
+			(at 254.3175 26.67 0)
+			(effects
+				(font
+					(size 1.27 1.27)
+				)
+			)
+		)
+		(property "Footprint" "PCM_Diode_SMD_AKL:D_SOD-523"
+			(at 254 30.48 0)
+			(effects
+				(font
+					(size 1.27 1.27)
+				)
+				(hide yes)
+			)
+		)
+		(property "Datasheet" "https://pdf.icgoo.net/productinfo/allpdf/e384d590-e1ec-3fe9-a3d3-7682eb2dfe94.pdf"
+			(at 254 30.48 0)
+			(effects
+				(font
+					(size 1.27 1.27)
+				)
+				(hide yes)
+			)
+		)
+		(property "Description" "SOD-523 Schottky diode, 30V, 200mA, Alternate KiCAD Library"
+			(at 254 30.48 0)
+			(effects
+				(font
+					(size 1.27 1.27)
+				)
+				(hide yes)
+			)
+		)
+		(pin "1"
+		)
+		(pin "2"
+		)
+		(instances
+			(project "rp2354a_micro_devboard"
+				(path "/2112ecc0-ac9a-4b37-bfed-d4d93ecb9ee7"
+					(reference "D2")
+					(unit 1)
+				)
+			)
+		)
